File: PROJET_SYSBEE/Sysbee/SIM800L.sch (KiCad schematic (older format))
At the start: 1 part

Commit message: placement et routage ok
Parts:
- GSM_SIM800L1: renamed from GSM_Module1; value SIM800L -> GSM_SIM800L
Changed lines of the file:
@@
 GSM SIM800L
 $Comp
-L Sysbee-rescue:SIM800L-sim800l GSM_Module1
+L Sysbee-rescue:SIM800L-sim800l GSM_SIM800L1
 U 1 1 6035DF8A
 P 6075 3575
-F 0 "GSM_Module1" H 6100 4462 60  0000 C CNN
-F 1 "SIM800L" H 6100 4356 60  0000 C CNN
+F 0 "GSM_SIM800L1" H 6100 4462 60  0000 C CNN
+F 1 "GSM_SIM800L" H 6100 4356 60  0000 C CNN
 F 2 "SIM800L:SIM800L" H 6075 3575 60  0001 C CNN
 F 3 "" H 6075 3575 60  0001 C CNN
